Commit message: fix: EKF/IMU tuning, hardware bridge remappings, sensor config, and cleanup
Squashed fixes and cleanup:
- Set high gyro yaw covariance so EKF trusts wheel odom for rotation
- Remove gyro bias compensation, publish raw gyro like v2
- Apply wheel direction to encoder tick deltas
- Fix hardware bridge topic routing and GPS topic remapping
- Fix navsat_to_absolute_pose datum reading from mowgli params
- Add configurable GPS antenna and IMU positions via mowgli_robot.yaml
- Remove magnetometer absolute heading hacks from EKF config
- Tune Nav2 speed to 0.3 m/s and enable collision detection
- Let ekf_map publish map->odom TF, disable SLAM TF broadcast
- Update launch files for slam_heading_node and localization changes
- Add map_odom_fuser_node build target (experimental, not launched)
- Update URDF and simulation model for sensor frame corrections

File: src/mowgli_bringup/urdf/mowgli.urdf.xacro (robot description, xacro)
@@ -24,4 +24,11 @@
   <xacro:arg name="lidar_z"   default="0.22"/>
   <xacro:arg name="lidar_yaw" default="0.0"/>
+  <xacro:arg name="imu_x"     default="0.0"/>
+  <xacro:arg name="imu_y"     default="0.0"/>
+  <xacro:arg name="imu_z"     default="0.095"/>
+  <xacro:arg name="imu_yaw"   default="0.0"/>
+  <xacro:arg name="gps_x"     default="0.0"/>
+  <xacro:arg name="gps_y"     default="0.0"/>
+  <xacro:arg name="gps_z"     default="0.20"/>
   <!-- ================================================================
        Properties
@@ -268,5 +275,5 @@
     <parent link="base_link"/>
     <child  link="imu_link"/>
-    <origin xyz="0 0 ${base_height/2}" rpy="0 0 0"/>
+    <origin xyz="$(arg imu_x) $(arg imu_y) $(arg imu_z)" rpy="0 0 $(arg imu_yaw)"/>
   </joint>
   <!-- ================================================================
@@ -299,6 +306,5 @@
     <parent link="base_link"/>
     <child  link="gps_link"/>
-    <!-- Mounted on top surface, centred -->
-    <origin xyz="0 0 ${base_height + 0.01}" rpy="0 0 0"/>
+    <origin xyz="$(arg gps_x) $(arg gps_y) $(arg gps_z)" rpy="0 0 0"/>
   </joint>
   <!-- ================================================================

Commit message: refactor: move base_link to rear wheel axis centre
Move base_link origin from chassis geometric centre to the centre of the
rear drive wheel axis, matching OpenMower convention. All sensor offsets
(lidar, IMU, GPS) updated relative to new origin. Chassis visual/collision
geometry uses configurable chassis_center_x parameter. Nav2 footprint
updated for asymmetric shape.

File: src/mowgli_bringup/urdf/mowgli.urdf.xacro (robot description, xacro)
@@ -20,9 +20,9 @@
        Configurable arguments (can be overridden via xacro command-line)
        ================================================================ -->
-  <xacro:arg name="lidar_x"   default="0.20"/>
+  <xacro:arg name="lidar_x"   default="0.38"/>
   <xacro:arg name="lidar_y"   default="0.0"/>
   <xacro:arg name="lidar_z"   default="0.22"/>
   <xacro:arg name="lidar_yaw" default="0.0"/>
-  <xacro:arg name="imu_x"     default="0.0"/>
+  <xacro:arg name="imu_x"     default="0.18"/>
   <xacro:arg name="imu_y"     default="0.0"/>
   <xacro:arg name="imu_z"     default="0.095"/>
@@ -31,4 +31,6 @@
   <xacro:arg name="gps_y"     default="0.0"/>
   <xacro:arg name="gps_z"     default="0.20"/>
+  <!-- Chassis geometry offset: distance from base_link (wheel axis) to chassis centre -->
+  <xacro:arg name="chassis_center_x" default="0.18"/>
   <!-- ================================================================
        Properties
@@ -42,11 +44,11 @@
   <xacro:property name="wheel_track"     value="0.40"/>  <!-- centre-to-centre -->
   <xacro:property name="wheel_mass"      value="0.5"/>
-  <!-- Rear wheels are offset behind base_link centre -->
-  <xacro:property name="wheel_x_offset"  value="-0.18"/>
+  <!-- Drive wheels at base_link (centre of rear wheel axis) -->
+  <xacro:property name="wheel_x_offset"  value="0.0"/>
   <!-- Front caster wheels (smaller) -->
   <xacro:property name="caster_radius"   value="0.03"/>
   <xacro:property name="caster_width"    value="0.03"/>
   <xacro:property name="caster_mass"     value="0.2"/>
-  <xacro:property name="caster_x_offset" value="0.22"/>
+  <xacro:property name="caster_x_offset" value="0.40"/>
   <xacro:property name="caster_track"    value="0.36"/>  <!-- centre-to-centre -->
   <xacro:property name="base_mass"       value="8.76"/>
@@ -106,9 +108,10 @@
   </joint>
   <!-- ================================================================
-       base_link  (geometric centre of chassis at wheel axle height)
+       base_link  (centre of rear drive wheel axis at wheel axle height)
        ================================================================ -->
   <link name="base_link">
     <visual>
-      <origin xyz="0 0 ${base_height/2}" rpy="0 0 0"/>
+      <!-- Chassis centre offset forward from wheel axis -->
+      <origin xyz="$(arg chassis_center_x) 0 ${base_height/2}" rpy="0 0 0"/>
       <geometry>
         <box size="${base_length} ${base_width} ${base_height}"/>
@@ -119,5 +122,5 @@
     </visual>
     <collision>
-      <origin xyz="0 0 ${base_height/2}" rpy="0 0 0"/>
+      <origin xyz="$(arg chassis_center_x) 0 ${base_height/2}" rpy="0 0 0"/>
       <geometry>
         <box size="${base_length} ${base_width} ${base_height}"/>
@@ -156,5 +159,5 @@
       <parent link="base_link"/>
       <child  link="${side}_wheel_link"/>
-      <!-- Rear drive wheels: offset behind base_link centre -->
+      <!-- Drive wheels at base_link origin -->
       <origin xyz="${wheel_x_offset} ${y_reflect * wheel_track/2} 0" rpy="0 0 0"/>
       <axis xyz="0 1 0"/>
@@ -242,6 +245,6 @@
     <parent link="base_link"/>
     <child  link="blade_link"/>
-    <!-- Blade disc centred under base, matching real robot -->
-    <origin xyz="0 0 ${-wheel_radius + 0.05}" rpy="0 0 0"/>
+    <!-- Blade disc centred under chassis -->
+    <origin xyz="$(arg chassis_center_x) 0 ${-wheel_radius + 0.05}" rpy="0 0 0"/>
     <axis xyz="0 0 1"/>
   </joint>

Commit message: fix: correct GPS antenna position and wheel track from OpenMower defaults
- gps_x: 0.0 -> 0.3 (antenna is 0.3m forward of wheel axis on YF500)
- wheel_track: 0.40 -> 0.325 (matches OpenMower OM_WHEEL_DISTANCE_M and
  kWheelBase in hardware_bridge)

File: src/mowgli_bringup/urdf/mowgli.urdf.xacro (robot description, xacro)
@@ -28,5 +28,5 @@
   <xacro:arg name="imu_z"     default="0.095"/>
   <xacro:arg name="imu_yaw"   default="0.0"/>
-  <xacro:arg name="gps_x"     default="0.0"/>
+  <xacro:arg name="gps_x"     default="0.3"/>
   <xacro:arg name="gps_y"     default="0.0"/>
   <xacro:arg name="gps_z"     default="0.20"/>
@@ -42,5 +42,5 @@
   <xacro:property name="wheel_radius"    value="0.04475"/>
   <xacro:property name="wheel_width"     value="0.04"/>
-  <xacro:property name="wheel_track"     value="0.40"/>  <!-- centre-to-centre -->
+  <xacro:property name="wheel_track"     value="0.325"/>  <!-- centre-to-centre -->
   <xacro:property name="wheel_mass"      value="0.5"/>
   <!-- Drive wheels at base_link (centre of rear wheel axis) -->

Commit message: refactor: all robot shape params from config, dynamic footprint
All URDF dimensions (chassis, wheels, casters, blade) now come from
mowgli_robot.yaml via xacro args. Nav2 footprint is computed at launch
time from chassis_length, chassis_width, chassis_center_x — no more
hardcoded coordinates. Different mower models only need config changes.

File: src/mowgli_bringup/urdf/mowgli.urdf.xacro (robot description, xacro)
@@ -31,29 +31,38 @@
   <xacro:arg name="gps_y"     default="0.0"/>
   <xacro:arg name="gps_z"     default="0.20"/>
-  <!-- Chassis geometry offset: distance from base_link (wheel axis) to chassis centre -->
+  <!-- Chassis shape (all from mowgli_robot.yaml via launch file) -->
+  <xacro:arg name="chassis_length"   default="0.54"/>
+  <xacro:arg name="chassis_width"    default="0.40"/>
+  <xacro:arg name="chassis_height"   default="0.19"/>
   <xacro:arg name="chassis_center_x" default="0.18"/>
-  <!-- ================================================================
-       Properties
-       ================================================================ -->
-  <xacro:property name="base_length"     value="0.54"/>
-  <xacro:property name="base_width"      value="0.40"/>
-  <xacro:property name="base_height"     value="0.19"/>
-  <!-- Rear drive wheels (from real URDF: diameter 0.0895m) -->
-  <xacro:property name="wheel_radius"    value="0.04475"/>
-  <xacro:property name="wheel_width"     value="0.04"/>
-  <xacro:property name="wheel_track"     value="0.325"/>  <!-- centre-to-centre -->
-  <xacro:property name="wheel_mass"      value="0.5"/>
-  <!-- Drive wheels at base_link (centre of rear wheel axis) -->
-  <xacro:property name="wheel_x_offset"  value="0.0"/>
-  <!-- Front caster wheels (smaller) -->
-  <xacro:property name="caster_radius"   value="0.03"/>
-  <xacro:property name="caster_width"    value="0.03"/>
-  <xacro:property name="caster_mass"     value="0.2"/>
-  <xacro:property name="caster_x_offset" value="0.40"/>
-  <xacro:property name="caster_track"    value="0.36"/>  <!-- centre-to-centre -->
-  <xacro:property name="base_mass"       value="8.76"/>
-  <xacro:property name="blade_radius"    value="0.09"/>
-  <xacro:property name="blade_height"    value="0.01"/>
-  <xacro:property name="blade_mass"      value="0.3"/>
+  <xacro:arg name="wheel_radius"     default="0.04475"/>
+  <xacro:arg name="wheel_width"      default="0.04"/>
+  <xacro:arg name="wheel_track"      default="0.325"/>
+  <xacro:arg name="wheel_x_offset"   default="0.0"/>
+  <xacro:arg name="caster_radius"    default="0.03"/>
+  <xacro:arg name="caster_track"     default="0.36"/>
+  <xacro:arg name="blade_radius"     default="0.09"/>
+  <!-- ================================================================
+       Properties (resolved from args — all shape from config)
+       ================================================================ -->
+  <xacro:property name="base_length"      value="$(arg chassis_length)"/>
+  <xacro:property name="base_width"       value="$(arg chassis_width)"/>
+  <xacro:property name="base_height"      value="$(arg chassis_height)"/>
+  <xacro:property name="chassis_cx"       value="$(arg chassis_center_x)"/>
+  <xacro:property name="wheel_radius"     value="$(arg wheel_radius)"/>
+  <xacro:property name="wheel_width"      value="$(arg wheel_width)"/>
+  <xacro:property name="wheel_track"      value="$(arg wheel_track)"/>
+  <xacro:property name="wheel_mass"       value="0.5"/>
+  <xacro:property name="wheel_x_offset"   value="$(arg wheel_x_offset)"/>
+  <xacro:property name="caster_radius"    value="$(arg caster_radius)"/>
+  <xacro:property name="caster_width"     value="0.03"/>
+  <xacro:property name="caster_mass"      value="0.2"/>
+  <!-- Casters near front edge of chassis -->
+  <xacro:property name="caster_x_offset"  value="${chassis_cx + base_length/2.0 - caster_radius}"/>
+  <xacro:property name="caster_track"     value="$(arg caster_track)"/>
+  <xacro:property name="base_mass"        value="8.76"/>
+  <xacro:property name="blade_radius"     value="$(arg blade_radius)"/>
+  <xacro:property name="blade_height"     value="0.01"/>
+  <xacro:property name="blade_mass"       value="0.3"/>
   <!-- Derived: base_link is wheel_radius above ground -->
   <xacro:property name="base_z_offset"   value="${wheel_radius}"/>
@@ -113,5 +122,5 @@
     <visual>
       <!-- Chassis centre offset forward from wheel axis -->
-      <origin xyz="$(arg chassis_center_x) 0 ${base_height/2}" rpy="0 0 0"/>
+      <origin xyz="${chassis_cx} 0 ${base_height/2}" rpy="0 0 0"/>
       <geometry>
         <box size="${base_length} ${base_width} ${base_height}"/>
@@ -122,5 +131,5 @@
     </visual>
     <collision>
-      <origin xyz="$(arg chassis_center_x) 0 ${base_height/2}" rpy="0 0 0"/>
+      <origin xyz="${chassis_cx} 0 ${base_height/2}" rpy="0 0 0"/>
       <geometry>
         <box size="${base_length} ${base_width} ${base_height}"/>
@@ -246,5 +255,5 @@
     <child  link="blade_link"/>
     <!-- Blade disc centred under chassis -->
-    <origin xyz="$(arg chassis_center_x) 0 ${-wheel_radius + 0.05}" rpy="0 0 0"/>
+    <origin xyz="${chassis_cx} 0 ${-wheel_radius + 0.05}" rpy="0 0 0"/>
     <axis xyz="0 0 1"/>
   </joint>
